Commit message: Fixed physics issues, and ros controls working

File: gazebo_cable_env/urdf/ur5e_hande.urdf.xacro (robot description, xacro)
@@ -21,5 +21,6 @@
     visual_parameters_file="$(find ur_description)/config/ur5e/visual_parameters.yaml"
   >
-    <origin xyz="0 0 0.45" rpy="0 0 0"/>
+    <!-- Table top is at z=0.425 (table center 0.4 + half height 0.025) -->
+    <origin xyz="0 0 0.425" rpy="0 0 0"/>
   </xacro:ur_robot>
   <!-- ============================================================ -->
@@ -220,15 +221,15 @@
   <xacro:property name="socket_height" value="0.004"/>  <!-- 4mm tall (thin) -->
   <xacro:property name="socket_depth" value="0.015"/>   <!-- 15mm deep -->
-  <xacro:property name="board_tilt" value="0.5"/>       <!-- ~29 degrees tilt -->
-  <!-- Board/fixture base - raised on a stand -->
+  <xacro:property name="board_tilt" value="0.3"/>       <!-- ~17 degrees tilt toward robot -->
+  <!-- Board/fixture base - on table -->
   <link name="board_stand">
     <visual>
-      <origin xyz="0 0 0.05"/>
-      <geometry><box size="0.08 0.08 0.1"/></geometry>
+      <origin xyz="0 0 0.04"/>
+      <geometry><box size="0.10 0.10 0.08"/></geometry>
       <material name="stand_dark"><color rgba="0.2 0.2 0.2 1"/></material>
     </visual>
     <collision>
-      <origin xyz="0 0 0.05"/>
-      <geometry><box size="0.08 0.08 0.1"/></geometry>
+      <origin xyz="0 0 0.04"/>
+      <geometry><box size="0.10 0.10 0.08"/></geometry>
     </collision>
     <inertial>
@@ -240,5 +241,6 @@
     <parent link="world"/>
     <child link="board_stand"/>
-    <origin xyz="0.5 -0.2 0.45" rpy="0 0 0"/>
+    <!-- Table top at z=0.425 -->
+    <origin xyz="0.5 -0.25 0.425" rpy="0 0 0"/>
   </joint>
   <!-- Tilted board/panel -->
@@ -260,5 +262,5 @@
     <child link="socket_board"/>
     <!-- Tilted forward so socket faces the robot -->
-    <origin xyz="0 0 0.1" rpy="${board_tilt} 0 0"/>
+    <origin xyz="0 0.02 0.08" rpy="${board_tilt} 0 0"/>
   </joint>
   <!-- USB-like socket housing (rectangular) -->
@@ -321,52 +323,31 @@
   </gazebo>
   <!-- ============================================================ -->
-  <!-- Deformable Cable (15 segments with 2-DOF joints)             -->
+  <!-- Deformable Cable (25 segments with 2-DOF joints)             -->
   <!-- ============================================================ -->
   <!-- Cable parameters - tuned for physics stability -->
   <xacro:property name="cable_radius" value="0.005"/>
-  <xacro:property name="cable_length" value="0.60"/>  <!-- 60cm long cable -->
-  <xacro:property name="num_segments" value="15"/>
+  <xacro:property name="cable_length" value="1.50"/>  <!-- 150cm long cable (3x original) -->
+  <xacro:property name="num_segments" value="25"/>
   <xacro:property name="segment_length" value="${cable_length / num_segments}"/>
-  <xacro:property name="segment_mass" value="0.02"/>  <!-- heavier for stability -->
-  <!-- Cable anchor mount (raised stand) -->
-  <link name="cable_mount_stand">
-    <visual>
-      <origin xyz="0 0 0.15"/>
-      <geometry><box size="0.06 0.06 0.3"/></geometry>
-      <material name="mount_grey"><color rgba="0.4 0.4 0.4 1"/></material>
-    </visual>
-    <collision>
-      <origin xyz="0 0 0.15"/>
-      <geometry><box size="0.06 0.06 0.3"/></geometry>
-    </collision>
-    <inertial>
-      <mass value="1.0"/>
-      <inertia ixx="1e-2" ixy="0" ixz="0" iyy="1e-2" iyz="0" izz="1e-3"/>
-    </inertial>
-  </link>
-  <joint name="cable_mount_stand_joint" type="fixed">
+  <xacro:property name="segment_mass" value="0.015"/>  <!-- lighter per segment for longer cable -->
+  <!-- Cable anchor point - directly on table, no tower -->
+  <link name="cable_anchor">
+    <visual>
+      <geometry><cylinder radius="0.03" length="0.02"/></geometry>
+      <material name="anchor_dark"><color rgba="0.2 0.2 0.2 1"/></material>
+    </visual>
+    <collision>
+      <geometry><cylinder radius="0.03" length="0.02"/></geometry>
+    </collision>
+    <inertial>
+      <mass value="0.3"/>
+      <inertia ixx="1e-4" ixy="0" ixz="0" iyy="1e-4" iyz="0" izz="1e-4"/>
+    </inertial>
+  </link>
+  <joint name="cable_anchor_joint" type="fixed">
     <parent link="world"/>
-    <child link="cable_mount_stand"/>
-    <origin xyz="0.2 0.4 0.45" rpy="0 0 0"/>
-  </joint>
-  <!-- Cable anchor point (on top of stand) -->
-  <link name="cable_anchor">
-    <visual>
-      <geometry><cylinder radius="0.025" length="0.02"/></geometry>
-      <material name="anchor_dark"><color rgba="0.2 0.2 0.2 1"/></material>
-    </visual>
-    <collision>
-      <geometry><cylinder radius="0.025" length="0.02"/></geometry>
-    </collision>
-    <inertial>
-      <mass value="0.2"/>
-      <inertia ixx="1e-5" ixy="0" ixz="0" iyy="1e-5" iyz="0" izz="1e-5"/>
-    </inertial>
-  </link>
-  <joint name="cable_anchor_joint" type="fixed">
-    <parent link="cable_mount_stand"/>
     <child link="cable_anchor"/>
-    <!-- On top of the stand, cable hangs down -->
-    <origin xyz="0 0 0.3" rpy="0 0 0"/>
+    <!-- Directly on table surface at z=0.425 + 0.01 (half anchor height) -->
+    <origin xyz="0.3 0.35 0.435" rpy="0 0 0"/>
   </joint>
   <!-- Cable segment macro with 2-DOF (roll + pitch) -->
@@ -425,5 +406,5 @@
     </gazebo>
   </xacro:macro>
-  <!-- Generate 15 cable segments -->
+  <!-- Generate 25 cable segments -->
   <xacro:cable_segment_2dof index="0" parent_link="cable_anchor" is_first="true"/>
   <xacro:cable_segment_2dof index="1" parent_link="cable_segment_0"/>
@@ -441,4 +422,14 @@
   <xacro:cable_segment_2dof index="13" parent_link="cable_segment_12"/>
   <xacro:cable_segment_2dof index="14" parent_link="cable_segment_13"/>
+  <xacro:cable_segment_2dof index="15" parent_link="cable_segment_14"/>
+  <xacro:cable_segment_2dof index="16" parent_link="cable_segment_15"/>
+  <xacro:cable_segment_2dof index="17" parent_link="cable_segment_16"/>
+  <xacro:cable_segment_2dof index="18" parent_link="cable_segment_17"/>
+  <xacro:cable_segment_2dof index="19" parent_link="cable_segment_18"/>
+  <xacro:cable_segment_2dof index="20" parent_link="cable_segment_19"/>
+  <xacro:cable_segment_2dof index="21" parent_link="cable_segment_20"/>
+  <xacro:cable_segment_2dof index="22" parent_link="cable_segment_21"/>
+  <xacro:cable_segment_2dof index="23" parent_link="cable_segment_22"/>
+  <xacro:cable_segment_2dof index="24" parent_link="cable_segment_23"/>
   <!-- USB-like rectangular connector (plug) at end of cable -->
   <!-- Connector dimensions match socket: 12mm x 4mm -->
@@ -464,5 +455,5 @@
   </link>
   <joint name="connector_joint" type="fixed">
-    <parent link="cable_segment_14"/>
+    <parent link="cable_segment_24"/>
     <child link="connector_grip"/>
     <origin xyz="0 0 ${segment_length}" rpy="0 0 0"/>

Commit message: Lot's of shit fixed in basic Gazebo sim

File: gazebo_cable_env/urdf/ur5e_hande.urdf.xacro (robot description, xacro)
@@ -38,5 +38,5 @@
       <plugin>gz_ros2_control/GazeboSimSystem</plugin>
     </hardware>
-    <!-- UR5e Arm Joints -->
+    <!-- UR5e Arm Joints - Starting in a lowered working position -->
     <joint name="shoulder_pan_joint">
       <command_interface name="position">
@@ -56,5 +56,5 @@
       </command_interface>
       <state_interface name="position">
-        <param name="initial_value">-1.5708</param>
+        <param name="initial_value">-2.0</param>
       </state_interface>
       <state_interface name="velocity"/>
@@ -67,5 +67,5 @@
       </command_interface>
       <state_interface name="position">
-        <param name="initial_value">0.0</param>
+        <param name="initial_value">1.5</param>
       </state_interface>
       <state_interface name="velocity"/>
@@ -78,5 +78,5 @@
       </command_interface>
       <state_interface name="position">
-        <param name="initial_value">-1.5708</param>
+        <param name="initial_value">-1.07</param>
       </state_interface>
       <state_interface name="velocity"/>
@@ -89,5 +89,5 @@
       </command_interface>
       <state_interface name="position">
-        <param name="initial_value">0.0</param>
+        <param name="initial_value">-1.5708</param>
       </state_interface>
       <state_interface name="velocity"/>
@@ -106,4 +106,5 @@
     </joint>
     <!-- Robotiq Hand-E Gripper Joints (both fingers for proper control) -->
+    <!-- Initial value 0.005 = gripper closed, holding the cable connector -->
     <joint name="hande_left_finger_joint">
       <command_interface name="position">
@@ -112,5 +113,5 @@
       </command_interface>
       <state_interface name="position">
-        <param name="initial_value">0.025</param>
+        <param name="initial_value">0.005</param>
       </state_interface>
       <state_interface name="velocity"/>
@@ -122,5 +123,5 @@
       </command_interface>
       <state_interface name="position">
-        <param name="initial_value">0.025</param>
+        <param name="initial_value">0.005</param>
       </state_interface>
       <state_interface name="velocity"/>
@@ -207,11 +208,12 @@
     </gazebo>
   </xacro:macro>
-  <!-- Camera positions: 90 degrees apart around wrist, pointing toward gripper -->
+  <!-- Camera positions: further from wrist, pointing toward gripper/target -->
+  <!-- Cameras mounted on wrist_3_link, positioned to view the gripper and workspace -->
   <xacro:wrist_camera name="camera_left" parent="wrist_3_link"
-                      xyz="0 0.05 0.02" rpy="0 0.4 -1.5708"/>
+                      xyz="0 0.10 0.0" rpy="0 0.7 -1.5708"/>
   <xacro:wrist_camera name="camera_bottom" parent="wrist_3_link"
-                      xyz="0.05 0 0.02" rpy="0 0.4 0"/>
+                      xyz="0.10 0 0.0" rpy="0 0.7 0"/>
   <xacro:wrist_camera name="camera_right" parent="wrist_3_link"
-                      xyz="0 -0.05 0.02" rpy="0 0.4 1.5708"/>
+                      xyz="0 -0.10 0.0" rpy="0 0.7 1.5708"/>
   <!-- ============================================================ -->
   <!-- Socket Board with USB-like rectangular slot                  -->
@@ -221,5 +223,5 @@
   <xacro:property name="socket_height" value="0.004"/>  <!-- 4mm tall (thin) -->
   <xacro:property name="socket_depth" value="0.015"/>   <!-- 15mm deep -->
-  <xacro:property name="board_tilt" value="0.3"/>       <!-- ~17 degrees tilt toward robot -->
+  <xacro:property name="board_tilt" value="0.0"/>       <!-- Straight up, no tilt -->
   <!-- Board/fixture base - on table -->
   <link name="board_stand">
@@ -324,31 +326,76 @@
   <!-- ============================================================ -->
   <!-- Deformable Cable (25 segments with 2-DOF joints)             -->
-  <!-- ============================================================ -->
-  <!-- Cable parameters - tuned for physics stability -->
+  <!-- Cable is attached to gripper, hangs down to anchor on table  -->
+  <!-- ============================================================ -->
+  <!-- Cable parameters -->
   <xacro:property name="cable_radius" value="0.005"/>
-  <xacro:property name="cable_length" value="1.50"/>  <!-- 150cm long cable (3x original) -->
+  <xacro:property name="cable_length" value="1.0"/>  <!-- 100cm cable -->
   <xacro:property name="num_segments" value="25"/>
   <xacro:property name="segment_length" value="${cable_length / num_segments}"/>
-  <xacro:property name="segment_mass" value="0.015"/>  <!-- lighter per segment for longer cable -->
-  <!-- Cable anchor point - directly on table, no tower -->
-  <link name="cable_anchor">
-    <visual>
-      <geometry><cylinder radius="0.03" length="0.02"/></geometry>
-      <material name="anchor_dark"><color rgba="0.2 0.2 0.2 1"/></material>
+  <xacro:property name="segment_mass" value="0.012"/>
+  <!-- USB-like rectangular connector (plug) dimensions -->
+  <xacro:property name="plug_width" value="0.011"/>
+  <xacro:property name="plug_height" value="0.003"/>
+  <xacro:property name="plug_length" value="0.018"/>
+  <!-- ============================================================ -->
+  <!-- Connector attached to gripper (between fingers)              -->
+  <!-- ============================================================ -->
+  <!-- Connector grip section (held by gripper) -->
+  <link name="connector_grip">
+    <visual>
+      <origin xyz="0 0 0.01"/>
+      <geometry><box size="0.016 0.012 0.02"/></geometry>
+      <material name="grip_orange"><color rgba="0.9 0.5 0.1 1"/></material>
     </visual>
     <collision>
-      <geometry><cylinder radius="0.03" length="0.02"/></geometry>
+      <origin xyz="0 0 0.01"/>
+      <geometry><box size="0.016 0.012 0.02"/></geometry>
     </collision>
     <inertial>
-      <mass value="0.3"/>
-      <inertia ixx="1e-4" ixy="0" ixz="0" iyy="1e-4" iyz="0" izz="1e-4"/>
-    </inertial>
-  </link>
-  <joint name="cable_anchor_joint" type="fixed">
-    <parent link="world"/>
-    <child link="cable_anchor"/>
-    <!-- Directly on table surface at z=0.425 + 0.01 (half anchor height) -->
-    <origin xyz="0.3 0.35 0.435" rpy="0 0 0"/>
-  </joint>
+      <mass value="0.02"/>
+      <origin xyz="0 0 0.01"/>
+      <inertia ixx="1e-5" ixy="0" ixz="0" iyy="1e-5" iyz="0" izz="1e-5"/>
+    </inertial>
+  </link>
+  <!-- Fixed joint attaching connector to gripper body (between fingers) -->
+  <joint name="connector_to_gripper_joint" type="fixed">
+    <parent link="hande_link"/>
+    <child link="connector_grip"/>
+    <!-- Position at finger height, centered between fingers -->
+    <origin xyz="0 0 0.12" rpy="0 0 0"/>
+  </joint>
+  <!-- USB-like plug tip (extends forward from connector) -->
+  <link name="cable_connector">
+    <visual>
+      <origin xyz="0 0 ${plug_length/2}"/>
+      <geometry><box size="${plug_width} ${plug_height} ${plug_length}"/></geometry>
+      <material name="connector_metal"><color rgba="0.75 0.75 0.78 1"/></material>
+    </visual>
+    <collision>
+      <origin xyz="0 0 ${plug_length/2}"/>
+      <geometry><box size="${plug_width} ${plug_height} ${plug_length}"/></geometry>
+    </collision>
+    <inertial>
+      <mass value="0.01"/>
+      <origin xyz="0 0 ${plug_length/2}"/>
+      <inertia ixx="1e-5" ixy="0" ixz="0" iyy="1e-5" iyz="0" izz="1e-5"/>
+    </inertial>
+  </link>
+  <joint name="connector_tip_joint" type="fixed">
+    <parent link="connector_grip"/>
+    <child link="cable_connector"/>
+    <origin xyz="0 0 0.02" rpy="0 0 0"/>
+  </joint>
+  <gazebo reference="cable_connector">
+    <mu1>0.5</mu1>
+    <mu2>0.5</mu2>
+  </gazebo>
+  <gazebo reference="connector_grip">
+    <mu1>1.0</mu1>
+    <mu2>1.0</mu2>
+  </gazebo>
+  <!-- ============================================================ -->
+  <!-- Cable segments - chain from connector outward to free end    -->
+  <!-- ============================================================ -->
   <!-- Cable segment macro with 2-DOF (roll + pitch) -->
   <xacro:macro name="cable_segment_2dof" params="index parent_link is_first:=false">
@@ -358,6 +405,6 @@
       <child link="cable_roll_link_${index}"/>
       <xacro:if value="${is_first}">
-        <!-- First segment: rotate 90deg so cable extends horizontally (along -Y) -->
-        <origin xyz="0 0 0.01" rpy="1.5708 0 0"/>
+        <!-- First segment: start behind connector, cable extends backward -->
+        <origin xyz="0 0 -0.01" rpy="${pi} 0 0"/>
       </xacro:if>
       <xacro:unless value="${is_first}">
@@ -365,11 +412,11 @@
       </xacro:unless>
       <axis xyz="1 0 0"/>
-      <dynamics damping="0.05" friction="0.01"/>
-    </joint>
-    <!-- Invisible roll link - needs real mass/inertia for stability -->
+      <dynamics damping="5.0" friction="0.1"/>
+    </joint>
+    <!-- Invisible roll link -->
     <link name="cable_roll_link_${index}">
       <inertial>
-        <mass value="0.005"/>
-        <inertia ixx="1e-5" ixy="0" ixz="0" iyy="1e-5" iyz="0" izz="1e-5"/>
+        <mass value="0.002"/>
+        <inertia ixx="1e-6" ixy="0" ixz="0" iyy="1e-6" iyz="0" izz="1e-6"/>
       </inertial>
     </link>
@@ -380,5 +427,5 @@
       <origin xyz="0 0 0" rpy="0 0 0"/>
       <axis xyz="0 1 0"/>
-      <dynamics damping="0.05" friction="0.01"/>
+      <dynamics damping="5.0" friction="0.1"/>
     </joint>
     <!-- Visible cable segment -->
@@ -399,13 +446,13 @@
       </inertial>
     </link>
-    <!-- Gazebo settings for cable segment -->
     <gazebo reference="cable_segment_${index}">
       <mu1>0.8</mu1>
       <mu2>0.8</mu2>
-      <self_collide>true</self_collide>
+      <self_collide>false</self_collide>
     </gazebo>
   </xacro:macro>
-  <!-- Generate 25 cable segments -->
-  <xacro:cable_segment_2dof index="0" parent_link="cable_anchor" is_first="true"/>
+  <!-- Generate 25 cable segments from connector outward -->
+  <!-- No initial pitch - let gravity naturally drape the cable -->
+  <xacro:cable_segment_2dof index="0" parent_link="connector_grip" is_first="true"/>
   <xacro:cable_segment_2dof index="1" parent_link="cable_segment_0"/>
   <xacro:cable_segment_2dof index="2" parent_link="cable_segment_1"/>
@@ -432,60 +479,26 @@
   <xacro:cable_segment_2dof index="23" parent_link="cable_segment_22"/>
   <xacro:cable_segment_2dof index="24" parent_link="cable_segment_23"/>
-  <!-- USB-like rectangular connector (plug) at end of cable -->
-  <!-- Connector dimensions match socket: 12mm x 4mm -->
-  <xacro:property name="plug_width" value="0.011"/>   <!-- slightly smaller than socket -->
-  <xacro:property name="plug_height" value="0.003"/>  <!-- slightly smaller than socket -->
-  <xacro:property name="plug_length" value="0.018"/>  <!-- insertion depth -->
-  <!-- Connector grip section (part that gripper holds) -->
-  <link name="connector_grip">
-    <visual>
-      <origin xyz="0 0 0.01"/>
-      <geometry><box size="0.016 0.012 0.02"/></geometry>
-      <material name="grip_orange"><color rgba="0.9 0.5 0.1 1"/></material>
+  <!-- Cable anchor/weight at free end - heavy to stay on table -->
+  <link name="cable_anchor">
+    <visual>
+      <geometry><cylinder radius="0.025" length="0.02"/></geometry>
+      <material name="anchor_dark"><color rgba="0.3 0.3 0.3 1"/></material>
     </visual>
     <collision>
-      <origin xyz="0 0 0.01"/>
-      <geometry><box size="0.016 0.012 0.02"/></geometry>
+      <geometry><cylinder radius="0.025" length="0.02"/></geometry>
     </collision>
     <inertial>
-      <mass value="0.02"/>
-      <origin xyz="0 0 0.01"/>
-      <inertia ixx="1e-5" ixy="0" ixz="0" iyy="1e-5" iyz="0" izz="1e-5"/>
-    </inertial>
-  </link>
-  <joint name="connector_joint" type="fixed">
+      <mass value="0.5"/>
+      <inertia ixx="1e-4" ixy="0" ixz="0" iyy="1e-4" iyz="0" izz="1e-4"/>
+    </inertial>
+  </link>
+  <joint name="cable_anchor_joint" type="fixed">
     <parent link="cable_segment_24"/>
-    <child link="connector_grip"/>
+    <child link="cable_anchor"/>
     <origin xyz="0 0 ${segment_length}" rpy="0 0 0"/>
   </joint>
-  <!-- USB-like plug tip (thin rectangular prong) -->
-  <link name="cable_connector">
-    <visual>
-      <origin xyz="0 0 ${plug_length/2}"/>
-      <geometry><box size="${plug_width} ${plug_height} ${plug_length}"/></geometry>
-      <material name="connector_metal"><color rgba="0.75 0.75 0.78 1"/></material>
-    </visual>
-    <collision>
-      <origin xyz="0 0 ${plug_length/2}"/>
-      <geometry><box size="${plug_width} ${plug_height} ${plug_length}"/></geometry>
-    </collision>
-    <inertial>
-      <mass value="0.01"/>
-      <origin xyz="0 0 ${plug_length/2}"/>
-      <inertia ixx="1e-5" ixy="0" ixz="0" iyy="1e-5" iyz="0" izz="1e-5"/>
-    </inertial>
-  </link>
-  <joint name="connector_tip_joint" type="fixed">
-    <parent link="connector_grip"/>
-    <child link="cable_connector"/>
-    <origin xyz="0 0 0.02" rpy="0 0 0"/>
-  </joint>
-  <gazebo reference="cable_connector">
-    <mu1>0.5</mu1>
-    <mu2>0.5</mu2>
-  </gazebo>
-  <gazebo reference="connector_grip">
-    <mu1>1.0</mu1>
-    <mu2>1.0</mu2>
+  <gazebo reference="cable_anchor">
+    <mu1>2.0</mu1>
+    <mu2>2.0</mu2>
   </gazebo>
 </robot>
