Commit message: env set up properly in isaac sim - moving onto RWM training with cams

File: rwm_ur5e/urdf/cable_rigid_isaac.urdf.xacro (robot description, xacro)
@@ -8,5 +8,5 @@
   <!-- Cable parameters -->
   <xacro:property name="cable_radius" value="0.005"/>
-  <xacro:property name="cable_length" value="0.9"/>
+  <xacro:property name="cable_length" value="0.45"/>
   <xacro:property name="num_segments" value="15"/>
   <xacro:property name="segment_length" value="${cable_length / num_segments}"/>
